Commit message: Upgrade robot's camera

File: src/my_robot/urdf/my_robot.xacro (robot description, xacro)
@@ -148,4 +148,11 @@
         </visual>
     </link>
+    <joint name="camera_optical_joint" type="fixed">
+        <origin xyz="0 0 0" rpy="-1.5707 0 -1.5707"/>
+        <parent link="camera"/>
+        <child link="camera_link_optical"/>
+    </joint>
+    <link name="camera_link_optical">
+    </link>
     <joint name="hokuyo_joint" type="fixed">
         <origin xyz="0.25 0.0 0.1" rpy="0.0 0.0 0.0" />
